File: StabTester/StabTester.kicad_sch (KiCad schematic)
At the start: 6 parts

Commit message: hehe
Parts:
- added MX1, MX2, MX3, MX4, MX5, MX6: MX-NoLED, mx-switches:CherryMX-1.00U, symbol pcb-rescue:MX-NoLED-MX_Alps_Hybrid
Changed lines of the file:
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@@
     )
+  )
+  (symbol (lib_id "pcb-rescue:MX-NoLED-MX_Alps_Hybrid") (at 120.015 77.47 0) (unit 1)
+    (in_bom yes) (on_board yes)
+    (property "Reference" "MX5" (id 0) (at 120.8532 71.8058 0)
+      (effects (font (size 1.524 1.524)))
+    )
+    (property "Value" "MX-NoLED" (id 1) (at 120.8532 73.6854 0)
+      (effects (font (size 0.508 0.508)))
+    )
+    (property "Footprint" "mx-switches:CherryMX-1.00U" (id 2) (at 104.14 78.105 0)
+      (effects (font (size 1.524 1.524)) hide)
+    )
+    (property "Datasheet" "" (id 3) (at 104.14 78.105 0)
+      (effects (font (size 1.524 1.524)) hide)
+    )
+    (pin "1")
+    (pin "2")
+  )
+  (symbol (lib_id "pcb-rescue:MX-NoLED-MX_Alps_Hybrid") (at 119.38 88.9 0) (unit 1)
+    (in_bom yes) (on_board yes)
+    (property "Reference" "MX2" (id 0) (at 120.2182 83.2358 0)
+      (effects (font (size 1.524 1.524)))
+    )
+    (property "Value" "MX-NoLED" (id 1) (at 120.2182 85.1154 0)
+      (effects (font (size 0.508 0.508)))
+    )
+    (property "Footprint" "mx-switches:CherryMX-1.00U" (id 2) (at 103.505 89.535 0)
+      (effects (font (size 1.524 1.524)) hide)
+    )
+    (property "Datasheet" "" (id 3) (at 103.505 89.535 0)
+      (effects (font (size 1.524 1.524)) hide)
+    )
+    (pin "1")
+    (pin "2")
+  )
+  (symbol (lib_id "pcb-rescue:MX-NoLED-MX_Alps_Hybrid") (at 119.38 123.19 0) (unit 1)
+    (in_bom yes) (on_board yes)
+    (property "Reference" "MX4" (id 0) (at 120.2182 117.5258 0)
+      (effects (font (size 1.524 1.524)))
+    )
+    (property "Value" "MX-NoLED" (id 1) (at 120.2182 119.4054 0)
+      (effects (font (size 0.508 0.508)))
+    )
+    (property "Footprint" "mx-switches:CherryMX-1.00U" (id 2) (at 103.505 123.825 0)
+      (effects (font (size 1.524 1.524)) hide)
+    )
+    (property "Datasheet" "" (id 3) (at 103.505 123.825 0)
+      (effects (font (size 1.524 1.524)) hide)
+    )
+    (pin "1")
+    (pin "2")
+  )
+  (symbol (lib_id "pcb-rescue:MX-NoLED-MX_Alps_Hybrid") (at 118.745 134.62 0) (unit 1)
+    (in_bom yes) (on_board yes)
+    (property "Reference" "MX1" (id 0) (at 119.5832 128.9558 0)
+      (effects (font (size 1.524 1.524)))
+    )
+    (property "Value" "MX-NoLED" (id 1) (at 119.5832 130.8354 0)
+      (effects (font (size 0.508 0.508)))
+    )
+    (property "Footprint" "mx-switches:CherryMX-1.00U" (id 2) (at 102.87 135.255 0)
+      (effects (font (size 1.524 1.524)) hide)
+    )
+    (property "Datasheet" "" (id 3) (at 102.87 135.255 0)
+      (effects (font (size 1.524 1.524)) hide)
+    )
+    (pin "1")
+    (pin "2")
   )
   (symbol (lib_id "Mechanical:MountingHole") (at 86.995 125.095 0) (unit 1)
@@
       (effects (font (size 1.27 1.27)) hide)
     )
+  )
+  (symbol (lib_id "pcb-rescue:MX-NoLED-MX_Alps_Hybrid") (at 119.38 111.76 0) (unit 1)
+    (in_bom yes) (on_board yes)
+    (property "Reference" "MX3" (id 0) (at 120.2182 106.0958 0)
+      (effects (font (size 1.524 1.524)))
+    )
+    (property "Value" "MX-NoLED" (id 1) (at 120.2182 107.9754 0)
+      (effects (font (size 0.508 0.508)))
+    )
+    (property "Footprint" "mx-switches:CherryMX-1.00U" (id 2) (at 103.505 112.395 0)
+      (effects (font (size 1.524 1.524)) hide)
+    )
+    (property "Datasheet" "" (id 3) (at 103.505 112.395 0)
+      (effects (font (size 1.524 1.524)) hide)
+    )
+    (pin "1")
+    (pin "2")
+  )
+  (symbol (lib_id "pcb-rescue:MX-NoLED-MX_Alps_Hybrid") (at 120.015 100.33 0) (unit 1)
+    (in_bom yes) (on_board yes)
+    (property "Reference" "MX6" (id 0) (at 120.8532 94.6658 0)
+      (effects (font (size 1.524 1.524)))
+    )
+    (property "Value" "MX-NoLED" (id 1) (at 120.8532 96.5454 0)
+      (effects (font (size 0.508 0.508)))
+    )
+    (property "Footprint" "mx-switches:CherryMX-1.00U" (id 2) (at 104.14 100.965 0)
+      (effects (font (size 1.524 1.524)) hide)
+    )
+    (property "Datasheet" "" (id 3) (at 104.14 100.965 0)
+      (effects (font (size 1.524 1.524)) hide)
+    )
+    (pin "1")
+    (pin "2")
   )
   (symbol (lib_id "Mechanical:MountingHole") (at 87.63 95.885 0) (unit 1)
@@
       (reference "H6") (unit 1) (value "MountingHole") (footprint "Mounting_Keyboard_Stabilizer:Stabilizer_Cherry_MX_8.00u")
     )
+    (path "/7306acad-0ce7-44a8-b068-b551a1dd918f"
+      (reference "MX1") (unit 1) (value "MX-NoLED") (footprint "mx-switches:CherryMX-1.00U")
+    )
+    (path "/5ecb09f2-8eba-49b5-979b-3cfbffecea24"
+      (reference "MX2") (unit 1) (value "MX-NoLED") (footprint "mx-switches:CherryMX-1.00U")
+    )
+    (path "/ca12c20d-eaae-40e9-b5e5-913deed6ccf3"
+      (reference "MX3") (unit 1) (value "MX-NoLED") (footprint "mx-switches:CherryMX-1.00U")
+    )
+    (path "/65cdb168-5123-42be-a1eb-85547716db59"
+      (reference "MX4") (unit 1) (value "MX-NoLED") (footprint "mx-switches:CherryMX-1.00U")
+    )
+    (path "/44d0e09f-e1dd-4b2d-9d7a-180654c8baa4"
+      (reference "MX5") (unit 1) (value "MX-NoLED") (footprint "mx-switches:CherryMX-1.00U")
+    )
+    (path "/ce6b7cd8-783b-49b6-9bb2-3cf6854f58eb"
+      (reference "MX6") (unit 1) (value "MX-NoLED") (footprint "mx-switches:CherryMX-1.00U")
+    )
   )

Commit message: added mounting holes'
Parts:
- added H10, H7, H8, H9: MountingHole, Mounting_Keyboard_Stabilizer:Stabilizer_Cherry_MX_6.25u, symbol Mechanical:MountingHole
